File: PCB/PartyLine80.kicad_pcb (KiCad board)
At the start: 2 copper layers, 100 x 120 mm, 191 parts, among them J1 Phones, J2 Key, J3 BNC, J4 2.1 mm Barrel Jack, Q1 2N4401, Q10 2N7000, Q11 2N7000, Q12 2N4403, Q13 2N7000, Q14 2N4401, Q15 2N4401, Q16 2N4401, Q17 2N7000, Q18 2N7000, Q19 2N7000, Q2 2N4401, Q20 2N4401, Q3 2N4401, Q4 2N4401, Q5 2N4401, Q6 2N4401, Q7 2N4401, Q8 2N4401, Q9 2N4403, T1 FT37-43 3T:21T, T2 FT37-43 3T:21T, T3 FT37-43 10T Trifilar, T4 FT37-43 10T Trifilar, T5 FT37-43 10T Bifilar, X1 3.582 MHz, X2 3.582 MHz, X3 3.582 MHz, X4 3.582 MHz, X5 3.582 MHz

Commit message: Party Line 80 PCB Rev B
Parts:
- removed the C27 at (99.4, 70.3)
- removed the D9 at (106.9, 37.1)
- removed the R33 at (79.8, 122.8)
- added C26: 560n Film, Capacitor_THT:C_Rect_L7.0mm_W2.5mm_P5.00mm, F.Cu at (80.5, 125.8)
- added C28: 1u, Capacitor_THT:CP_Radial_D5.0mm_P2.50mm, F.Cu at (138.2, 51.1)
- added D15: 1N5237B, EtherkitKicadLibrary:D_DO-35_SOD27_P7.62mm_Horizontal, F.Cu at (109.7, 45.7)
- added L2: T37-2 22T, EtherkitKicadLibrary:T37-V, F.Cu at (143.5, 78.6)
- added R62: 1k, Resistor_THT:R_Axial_DIN0207_L6.3mm_D2.5mm_P2.54mm_Vertical, F.Cu at (102.5, 42.1)
- added TP14: +3.3V, TestPoint:TestPoint_THTPad_D2.0mm_Drill1.0mm, F.Cu at (113.9, 38.2)
- C16: value 100n -> 1u Film
- C18: value 1u -> 1u Film
- C25: value 10u -> 1u
- C27: renamed from C26; value 100n -> 560n Film
- D10: footprint Diode_THT:D_DO-35_SOD27_P7.62mm_Horizontal -> EtherkitKicadLibrary:D_DO-35_SOD27_P7.62mm_Horizontal
- moved D10 19.6 mm to (105.7, 45.7)
- moved R31 19.5 mm to (86.8, 135.9), turned to 0 degrees
- moved C30 11.9 mm to (145.1, 84.1)
- moved TP9 10.7 mm to (137.9, 87.6)
- moved C39 9.50 mm to (99.4, 70.3)
- moved R40 8.76 mm to (131.9, 49.2)
- moved R45 8.55 mm to (125.3, 51.2)
- moved R41 8.04 mm to (119.8, 51.2)
- moved TP6 6.15 mm to (113.9, 44.0)
- moved TP13 3.18 mm to (142.6, 91.1)
- moved Q11 1.73 mm to (78.6, 115.7)
- moved R18 0.90 mm to (123.9, 139.0)
- moved Q10 0.74 mm to (87.6, 115.7)
- moved TP7 0.50 mm to (98.3, 43.7)
- renumbered C15 to C13, C13 to C14, C14 to C15, C28 to C29, C29 to C30, C30 to C31, C31 to C32, C32 to C33, C33 to C34, C34 to C35, C35 to C36, C36 to C37, C37 to C38, C38 to C39, C39 to C40, C40 to C41, C41 to C42, C42 to C43, C43 to C44, C44 to C45, C45 to C46, C46 to C47, C47 to C48, C48 to C49, C49 to C50, C50 to C51, C51 to C52, C52 to C53, C53 to C54, D15 to D9, L2 to L3, L3 to L4, L4 to L5, L5 to L6, L6 to L7, L7 to L8, L8 to L9, R34 to R33, R35 to R34, R36 to R35, R37 to R36, R38 to R37, R39 to R38, R40 to R39, R41 to R40, R42 to R41, R43 to R42, R44 to R43, R45 to R44, R46 to R45, R47 to R46, R48 to R47, R49 to R48, R50 to R49, R54 to R50, R55 to R54, R56 to R55, R57 to R56, R58 to R57, R59 to R58, R60 to R59, R61 to R60, R62 to R61, TP10 to TP1, TP3 to TP10, TP8 to TP11, TP4 to TP12, TP5 to TP13, TP9 to TP2, TP11 to TP3, TP12 to TP4, TP13 to TP5, TP2 to TP8, TP1 to TP9
Connections:
- C24 pad 2: Net-(Q10-D) -> Net-(Q10-S)
- C27 pad 1: Net-(Q11-S) -> Net-(C26-Pad1)
- C30 pad 1: Net-(C29-Pad1) -> Net-(C30-Pad1)
- C34 pad 2: Net-(Q13-D) -> Net-(Q15-B)
- J1 pad R: Net-(Q11-S) -> Net-(C26-Pad1)
- J1 pad T: Net-(Q11-S) -> Net-(C26-Pad1)
- Q10 pad 1: GND -> Net-(Q10-S)
- Q10 pad 2: +12V K -> Net-(D7-A)
- Q14 pad 2: Net-(Q14-B) -> TX LO
- Q15 pad 2: Net-(Q13-D) -> Net-(Q15-B)
- R31 pad 1: +12V K -> Net-(D7-A)
- R31 pad 2: GND -> +3.3V
- R34 pad 1: Net-(D10-K) -> +3.3V
- R36 pad 2: Net-(Q14-B) -> TX LO
- R37 pad 1: Net-(Q14-B) -> TX LO
- R40 pad 1: Net-(D10-K) -> Net-(R40-Pad1)
- R40 pad 2: Net-(Q13-D) -> Net-(Q15-B)
- R41 pad 1: Net-(Q13-D) -> Net-(Q15-B)
- R44 pad 2: Net-(D9-K) -> Net-(D10-K)
- R45 pad 1: Net-(D10-K) -> Net-(R40-Pad1)
- R47 pad 1: Net-(D9-K) -> Net-(D10-K)
- R50 pad 2: Net-(D10-K) -> Net-(R40-Pad1)
- R51 pad 1: Net-(D10-K) -> Net-(R40-Pad1)
- X5 pad 1: Net-(C29-Pad1) -> Net-(Q13-D)
- X5 pad 2: Net-(Q13-D) -> Net-(Q15-B)
Routing:
- net +3.3V: track 0.00 -> 175.3 mm, vias 0 -> 1
- net Net-(Q15-B): track 0.00 -> 44.8 mm
- net Net-(D10-K): track 54.2 -> 11.2 mm
- net Net-(R40-Pad1): track 0.00 -> 34.7 mm
- net Net-(Q11-S): track 30.8 -> 5.90 mm
- net Net-(C26-Pad1): track 0.00 -> 24.0 mm
- net +12V: track 284.4 -> 261.1 mm
- net Net-(Q14-B): track 21.1 -> 0.00 mm
- net +12V K: track 158.8 -> 138.8 mm, vias 0 -> 2
- net Net-(Q13-D): track 47.4 -> 27.7 mm
- net TX LO: track 9.60 -> 28.3 mm
- net Net-(D9-K): track 14.5 -> 0.00 mm
- net Net-(Q10-S): track 0.00 -> 13.3 mm
- net Net-(D7-A): track 21.8 -> 33.7 mm
- net Net-(D8-A): track 12.6 -> 22.3 mm
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Other:
- board text added: "Rev B"
- board text removed: "Rev A"
