File: PCB/rx.kicad_sch (KiCad schematic)
At the start: 91 parts, among them J1 Phones, Q1 2N4401, Q10 2N7000, Q11 2N7000, Q2 2N4401, Q3 2N4401, Q4 2N4401, Q5 2N4401, Q6 2N4401, Q7 2N4401, Q8 2N4401, Q9 2N4403, T1 FT37-43 10T Trifilar, T1 FT37-43 3T:21T, T2 FT37-43 10T Trifilar, T2 FT37-43 3T:21T, X1 3.582 MHz, X2 3.582 MHz, X3 3.582 MHz, X4 3.582 MHz

Commit message: Add basic build instructions
Parts:
- renumbered TP8 to TP10, TP8 to TP11, TP8 to TP12, TP8 to TP9
Changed lines of the file:
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@@
   (symbol (lib_id "Connector:TestPoint") (at 68.58 96.52 0) (unit 1)
     (in_bom yes) (on_board yes) (dnp no) (fields_autoplaced)
-    (property "Reference" "TP8" (at 71.12 91.948 0)
+    (property "Reference" "TP11" (at 71.12 91.948 0)
       (effects (font (size 1.27 1.27)) (justify left))
     )
@@
     (instances
       (project "PartyLine80"
-        (path "/b5844e62-3e3b-42e9-bb77-207602f5ec8e/b7bb4922-3f83-4fe7-b552-685e81511d4b"
-          (reference "TP8") (unit 1)
-        )
         (path "/b5844e62-3e3b-42e9-bb77-207602f5ec8e/10258d8b-bf3e-4721-8c4f-caff16e423d7"
           (reference "TP11") (unit 1)
@@
   (symbol (lib_id "Connector:TestPoint") (at 15.24 60.96 0) (unit 1)
     (in_bom yes) (on_board yes) (dnp no) (fields_autoplaced)
-    (property "Reference" "TP8" (at 17.78 56.388 0)
+    (property "Reference" "TP10" (at 17.78 56.388 0)
       (effects (font (size 1.27 1.27)) (justify left))
     )
@@
     (instances
       (project "PartyLine80"
-        (path "/b5844e62-3e3b-42e9-bb77-207602f5ec8e/b7bb4922-3f83-4fe7-b552-685e81511d4b"
-          (reference "TP8") (unit 1)
-        )
         (path "/b5844e62-3e3b-42e9-bb77-207602f5ec8e/10258d8b-bf3e-4721-8c4f-caff16e423d7"
           (reference "TP10") (unit 1)
@@
   (symbol (lib_id "Connector:TestPoint") (at 138.176 100.584 0) (unit 1)
     (in_bom yes) (on_board yes) (dnp no) (fields_autoplaced)
-    (property "Reference" "TP8" (at 139.7 96.012 0)
+    (property "Reference" "TP12" (at 139.7 96.012 0)
       (effects (font (size 1.27 1.27)) (justify left))
     )
@@
     (instances
       (project "PartyLine80"
-        (path "/b5844e62-3e3b-42e9-bb77-207602f5ec8e/b7bb4922-3f83-4fe7-b552-685e81511d4b"
-          (reference "TP8") (unit 1)
-        )
         (path "/b5844e62-3e3b-42e9-bb77-207602f5ec8e/10258d8b-bf3e-4721-8c4f-caff16e423d7"
           (reference "TP12") (unit 1)
@@
   (symbol (lib_id "Connector:TestPoint") (at 58.42 27.94 0) (unit 1)
     (in_bom yes) (on_board yes) (dnp no) (fields_autoplaced)
-    (property "Reference" "TP8" (at 60.96 23.368 0)
+    (property "Reference" "TP9" (at 60.96 23.368 0)
       (effects (font (size 1.27 1.27)) (justify left))
     )
@@
     (instances
       (project "PartyLine80"
-        (path "/b5844e62-3e3b-42e9-bb77-207602f5ec8e/b7bb4922-3f83-4fe7-b552-685e81511d4b"
-          (reference "TP8") (unit 1)
-        )
         (path "/b5844e62-3e3b-42e9-bb77-207602f5ec8e/10258d8b-bf3e-4721-8c4f-caff16e423d7"
           (reference "TP9") (unit 1)

Commit message: Party Line 80 PCB Rev B
Parts:
- removed R31: 100k, Resistor_THT:R_Axial_DIN0207_L6.3mm_D2.5mm_P2.54mm_Vertical, symbol Device:R_US
- added C26: 560n Film, Capacitor_THT:C_Rect_L7.0mm_W2.5mm_P5.00mm, symbol Device:C_Small
- C16: value 100n -> 1u Film
- C18: value 1u -> 1u Film
- C25: value 10u -> 1u
- C27: renamed from C26; value 100n -> 560n Film
- renumbered C15 to C13, C13 to C14, C14 to C15, R33 to R31, TP10 to TP1, TP9 to TP2, TP11 to TP3, TP12 to TP4
Connections:
- net +12V K is gone; now on an unnamed net: Q10.2 (G)
- net +12V: no longer R31.2
- net GND: no longer Q10.1 (S)
- net at Q10.3 (D), Q11.3 (D): no longer C24.2
- net at C27.1, J1.R, J1.T: now also C26.1; no longer Q11.1 (S)
- new net: C26.2, Q11.1 (S)
- new net: C24.2, Q10.1 (S)
- new net +3.3V: R31.2
Other:
- moved on the sheet: C24, C25, D7, Q10, Q11, R31
